File: kicad/lampe.kicad_sch (KiCad schematic)
At the start: 81 parts, among them U1 WeMos_D1_mini, X1 SW_Push, Y1 SW_Push

Commit message: +transistor and led footprint edit => spread the legs... euh
Parts:
- B13, B14, G13, G14, R14: footprint Resistor_THT:R_Axial_DIN0207_L6.3mm_D2.5mm_P2.54mm_Vertical -> Resistor_THT:R_Axial_DIN0207_L6.3mm_D2.5mm_P10.16mm_Horizontal
- D1, D10, D11, D12, D13, D14, D15, D16, D17, D2, D3, D4, D5, D6, D7, D8, D9: footprint LED_THT:LED_D5.0mm-4_RGB -> pierre:LED_RAGB_5mm_v2
- QB1, QG1, QR1: footprint Package_TO_SOT_THT:TO-92_Inline -> pierre:Q_NPN_EBC_TO-92_v2
